File: ft4232.sch (KiCad schematic (older format))
At the start: 23 parts, among them J301 Conn_01x12, J302 Conn_01x12, J303 Conn_01x12, J304 Conn_01x12, U301 FT4232H, U302 93CxxA, Y301 Crystal

Commit message: Revision 2
Parts:
- removed U302: 93CxxA, Package_DIP:DIP-8_W7.62mm_Socket, symbol Memory_EEPROM:93CxxA
- added U302: 93CxxC, Package_DIP:DIP-8_W7.62mm_Socket, symbol Memory_EEPROM:93CxxC
Connections:
- net +3V3: now also L301.1, L302.1, U302.6 (ORG), U302.8 (VCC)
- net GND: now also U302.5 (GND)
- net at C301.1, C302.1, C305.1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: no longer L301.1, L302.1
- net UARTSW_TX_C: now reaches J304.3 (Pin_3), U301.48 (DDBUS0)
- net UARTSW_RX_C: now reaches J304.4 (Pin_4), U301.52 (DDBUS1)
- net at R304.1, U301.61 (EEDATA): now also U302.3 (DI)
- net at R302.2, U301.62 (EECLK): now also U302.2 (SCLK)
- net at R303.2, U301.63 (EECS): now also U302.1 (CS)
- net at R301.2, R304.2: now also U302.4 (DO)
Changed lines of the file:
@@
 $EndComp
 Wire Wire Line
-	4000 1000 4000 1250
+	4000 1000 4000 1050
 Wire Wire Line
 	4000 1600 4100 1600
@@
 	2600 2100 2350 2100
 Wire Wire Line
-	2350 2100 2350 900
-Wire Wire Line
-	2350 900  3050 900
-Wire Wire Line
-	3800 900  3800 1600
-Wire Wire Line
 	3600 1600 3700 1600
-Connection ~ 3800 1600
 Connection ~ 3700 1600
 Wire Wire Line
@@
 	1    0    0    -1
 $EndComp
-Connection ~ 3050 900
-Wire Wire Line
-	3050 900  3400 900
 $Comp
 L Device:L L302
@@
 	1    0    0    -1
 $EndComp
-Connection ~ 3400 900
-Wire Wire Line
-	3400 900  3800 900
 Wire Wire Line
 	3400 1200 3400 1400
@@
 	8800 4850 8800 3650
 Wire Wire Line
-	8800 3650 10300 3650
-Wire Wire Line
 	8900 3750 8900 4900
 Wire Wire Line
@@
 Wire Wire Line
 	7600 4900 7600 4700
-Wire Wire Line
-	8900 3750 10300 3750
 Wire Wire Line
 	7550 4800 7550 4950
@@
 F 3 "" H 2150 3500 50  0001 C CNN
 	1    2150 3500
-	1    0    0    -1
-$EndComp
-$Comp
-L Memory_EEPROM:93CxxA U302
-U 1 1 61BE30C5
-P 1000 4450
-F 0 "U302" H 1000 4931 50  0000 C CNN
-F 1 "93CxxA" H 1000 4840 50  0000 C CNN
-F 2 "Package_DIP:DIP-8_W7.62mm_Socket" H 1000 4450 50  0001 C CNN
-F 3 "http://ww1.microchip.com/downloads/en/DeviceDoc/20001749K.pdf" H 1000 4450 50  0001 C CNN
-	1    1000 4450
 	1    0    0    -1
 $EndComp
@@
 	1400 3150 950  3150
 Connection ~ 950  3150
+Wire Wire Line
+	3700 1600 3700 700
+Wire Wire Line
+	3700 700  2350 700
+Wire Wire Line
+	2350 700  2350 2100
+Wire Wire Line
+	3050 900  3400 900
+Wire Wire Line
+	3400 900  3850 900
+Wire Wire Line
+	3850 900  3850 1050
+Wire Wire Line
+	3850 1050 4000 1050
+Connection ~ 3400 900
+Connection ~ 4000 1050
+Wire Wire Line
+	4000 1050 4000 1250
+Wire Wire Line
+	8800 3650 9550 3650
+Wire Wire Line
+	8900 3750 9600 3750
+Wire Wire Line
+	9550 3650 9550 3400
+Wire Wire Line
+	9550 3400 9450 3400
+Connection ~ 9550 3650
+Wire Wire Line
+	9550 3650 10300 3650
+Wire Wire Line
+	9450 3300 9600 3300
+Wire Wire Line
+	9600 3300 9600 3750
+Connection ~ 9600 3750
+Wire Wire Line
+	9600 3750 10300 3750
+Text GLabel 9450 3400 0    50   Input ~ 0
+UARTSW_TX_C
+Text GLabel 9450 3300 0    50   Input ~ 0
+UARTSW_RX_C
+$Comp
+L Memory_EEPROM:93CxxC U302
+U 1 1 622876DE
+P 1000 4450
+F 0 "U302" H 1100 4800 50  0000 C CNN
+F 1 "93CxxC" H 1200 4700 50  0000 C CNN
+F 2 "Package_DIP:DIP-8_W7.62mm_Socket" H 1000 4450 50  0001 C CNN
+F 3 "http://ww1.microchip.com/downloads/en/DeviceDoc/20001749K.pdf" H 1000 4450 50  0001 C CNN
+	1    1000 4450
+	1    0    0    -1
+$EndComp
+Wire Wire Line
+	600  4450 550  4450
+Wire Wire Line
+	550  4450 550  4150
+Wire Wire Line
+	550  4150 1000 4150
+Connection ~ 1000 4150
 $EndSCHEMATC
