File: usb_hub.sch (KiCad schematic (older format))
At the start: 25 parts, among them J201 Conn_02x04_Top_Bottom, J202 8P8C_LED_Shielded, U101 LAN9514

Commit message: Revision 2
Parts:
- added C206, C207, C208, C209: .1uF, Capacitor_SMD:C_0603_1608Metric_Pad1.08x0.95mm_HandSolder, symbol Device:C
- added D201, D202: LED, LED_SMD:LED_0603_1608Metric_Pad1.05x0.95mm_HandSolder, symbol Device:LED
- added J203, J205, J206, J207, J208: Conn_01x04, Connector_PinHeader_2.54mm:PinHeader_1x04_P2.54mm_Vertical, symbol Connector_Generic:Conn_01x04
- added J204: Conn_01x08, Connector_PinHeader_2.54mm:PinHeader_2x04_P2.54mm_Vertical, symbol Connector_Generic:Conn_01x08
- added R214, R215, R216, R217, R218, R219, R220, R221: 680k, Resistor_SMD:R_0603_1608Metric_Pad0.98x0.95mm_HandSolder, symbol Device:R
- added R222, R223: 470, Resistor_SMD:R_0603_1608Metric_Pad0.98x0.95mm_HandSolder, symbol Device:R
- added U201: SN74CBT3253, Package_SO:SOIC-16_3.9x9.9mm_P1.27mm, symbol Analog_Switch:SN74CBT3253
- added U202: PCF8574, Package_SO:SOIC-16W_7.5x10.3mm_P1.27mm, symbol Interface_Expansion:PCF8574
- J202: symbol custom:8P8C_LED_Shielded -> iotether-rescue:8P8C_LED_Shielded-custom
Connections:
- net +3V3: now also J206.1 (Pin_1), J208.1 (Pin_1), R216.1, R217.1, R220.1, R221.1, R222.1, R223.1; no longer R206.1, R207.1, R208.1, R209.1, R212.1
- net +5V: now also J205.1 (Pin_1), J207.1 (Pin_1), R214.1, R215.1, R218.1, R219.1, U201.16 (VCC)
- net GND: now also C206.2, C207.2, C208.2, C209.2, J203.2 (Pin_2), J204.8 (Pin_8), J205.4 (Pin_4), J206.4 (Pin_4), J207.4 (Pin_4), J208.4 (Pin_4), U201.1 (1~OE), U201.15 (2~OE), U201.8 (GND), U202.1 (A0), U202.3 (A2), U202.8 (VSS)
- new net: J204.5 (Pin_5), U202.10 (P5)
- new net: J204.6 (Pin_6), U202.11 (P6)
- new net: J204.7 (Pin_7), U202.12 (P7)
- new net: J204.2 (Pin_2), U202.6 (P2)
- new net: J204.3 (Pin_3), U202.7 (P3)
- new net: J204.4 (Pin_4), U202.9 (P4)
- new net: D201.2 (A), R222.2
- new net: D202.2 (A), R223.2
- new net +3.3VA: C206.1, C207.1, C208.1, C209.1, R206.1, R207.1, R208.1, R209.1, R212.1
- new net EXT_PWR: J203.1 (Pin_1), J204.1 (Pin_1), U202.16 (VDD), U202.2 (A1)
- new net EXT_SCL: J203.4 (Pin_4), U202.14 (SCL)
- new net EXT_SDA: J203.3 (Pin_3), U202.15 (SDA)
- new net SW0: D201.1 (K), U201.14 (S0), U202.4 (P0)
- new net SW1: D202.1 (K), U201.2 (S1), U202.5 (P1)
- new net UARTSW_RX_C: U201.7 (1A)
- new net UARTSW_TX_C: U201.9 (2A)
- new net USW_RX_E1: J205.2 (Pin_2), R215.2, U201.6 (1B1)
- new net USW_RX_E2: J207.2 (Pin_2), R219.2, U201.5 (1B2)
- new net USW_RX_E3: J206.2 (Pin_2), R217.2, U201.4 (1B3)
- new net USW_RX_E4: J208.2 (Pin_2), R221.2, U201.3 (1B4)
- new net USW_TX_E1: J205.3 (Pin_3), R214.2, U201.10 (2B1)
- new net USW_TX_E2: J207.3 (Pin_3), R218.2, U201.11 (2B2)
- new net USW_TX_E3: J206.3 (Pin_3), R216.2, U201.12 (2B3)
- new net USW_TX_E4: J208.3 (Pin_3), R220.2, U201.13 (2B4)
Other:
- moved on the sheet: JP201, JP202, JP203, JP204
