File: ft4232.kicad_sch (KiCad schematic)
At the start: 23 parts, among them J301 Conn_01x12, J302 Conn_01x12, J303 Conn_01x12, J304 Conn_01x12, U301 FT4232H, U302 93CxxC, Y301 Crystal

Commit message: Add i2c_sampler, update to revision 3
Parts:
- R304: footprint Resistor_SMD:R_0603_1608Metric_Pad1.05x0.95mm_HandSolder -> Resistor_SMD:R_0603_1608Metric_Pad0.98x0.95mm_HandSolder
Connections:
- net ATM_RX: now reaches J302.3 (Pin_3), U301.38 (CDBUS0)
- net ATM_TX: now reaches J302.4 (Pin_4), U301.39 (CDBUS1)
- net ATM_DTR: now reaches J302.7 (Pin_7), U301.43 (CDBUS4)
Changed lines of the file:
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@@
   (junction (at 86.36 22.86) (diameter 0) (color 0 0 0 0)
   )
+  (junction (at 153.67 96.52) (diameter 0) (color 0 0 0 0)
+  )
+  (junction (at 170.18 93.98) (diameter 0) (color 0 0 0 0)
+  )
   (junction (at 91.44 149.86) (diameter 0) (color 0 0 0 0)
   )
@@
   (junction (at 101.6 40.64) (diameter 0) (color 0 0 0 0)
   )
+  (junction (at 139.7 104.14) (diameter 0) (color 0 0 0 0)
+  )
   (junction (at 101.6 26.67) (diameter 0) (color 0 0 0 0)
   )
@@
     (stroke (width 0) (type default) (color 0 0 0 0))
   )
-  (wire (pts (xy 127 96.52) (xy 201.93 96.52))
+  (wire (pts (xy 127 96.52) (xy 153.67 96.52))
     (stroke (width 0) (type default) (color 0 0 0 0))
   )
@@
     (stroke (width 0) (type default) (color 0 0 0 0))
   )
+  (wire (pts (xy 153.67 91.44) (xy 153.67 96.52))
+    (stroke (width 0) (type default) (color 0 0 0 0))
+  )
   (wire (pts (xy 181.61 62.23) (xy 210.82 62.23))
     (stroke (width 0) (type default) (color 0 0 0 0))
@@
     (stroke (width 0) (type default) (color 0 0 0 0))
   )
+  (wire (pts (xy 170.18 91.44) (xy 170.18 93.98))
+    (stroke (width 0) (type default) (color 0 0 0 0))
+  )
   (wire (pts (xy 59.69 119.38) (xy 59.69 114.3))
     (stroke (width 0) (type default) (color 0 0 0 0))
@@
     (stroke (width 0) (type default) (color 0 0 0 0))
   )
-  (wire (pts (xy 127 104.14) (xy 201.93 104.14))
+  (wire (pts (xy 127 104.14) (xy 139.7 104.14))
     (stroke (width 0) (type default) (color 0 0 0 0))
   )
@@
     (stroke (width 0) (type default) (color 0 0 0 0))
   )
-  (wire (pts (xy 127 93.98) (xy 201.93 93.98))
+  (wire (pts (xy 127 93.98) (xy 170.18 93.98))
     (stroke (width 0) (type default) (color 0 0 0 0))
   )
@@
     (stroke (width 0) (type default) (color 0 0 0 0))
   )
+  (wire (pts (xy 170.18 93.98) (xy 201.93 93.98))
+    (stroke (width 0) (type default) (color 0 0 0 0))
+  )
   (wire (pts (xy 229.87 128.27) (xy 229.87 102.87))
     (stroke (width 0) (type default) (color 0 0 0 0))
@@
     (stroke (width 0) (type default) (color 0 0 0 0))
   )
+  (wire (pts (xy 139.7 104.14) (xy 201.93 104.14))
+    (stroke (width 0) (type default) (color 0 0 0 0))
+  )
   (wire (pts (xy 151.13 43.18) (xy 146.05 43.18))
     (stroke (width 0) (type default) (color 0 0 0 0))
@@
     (stroke (width 0) (type default) (color 0 0 0 0))
   )
+  (wire (pts (xy 153.67 96.52) (xy 201.93 96.52))
+    (stroke (width 0) (type default) (color 0 0 0 0))
+  )
   (wire (pts (xy 135.89 35.56) (xy 135.89 45.72))
     (stroke (width 0) (type default) (color 0 0 0 0))
@@
     (stroke (width 0) (type default) (color 0 0 0 0))
   )
+  (wire (pts (xy 139.7 91.44) (xy 139.7 104.14))
+    (stroke (width 0) (type default) (color 0 0 0 0))
+  )
   (wire (pts (xy 33.02 55.88) (xy 41.91 55.88))
     (stroke (width 0) (type default) (color 0 0 0 0))
@@
   (wire (pts (xy 151.13 53.34) (xy 127 53.34))
     (stroke (width 0) (type default) (color 0 0 0 0))
+  )
+  (global_label "ATM_DTR" (shape input) (at 139.7 91.44 0) (fields_autoplaced)
+    (effects (font (size 1.27 1.27)) (justify left))
+    (property "Intersheet References" "${INTERSHEET_REFS}" (id 0) (at 150.0071 91.3606 0)
+      (effects (font (size 1.27 1.27)) (justify left) hide)
+    )
   )
   (global_label "UARTSW_TX_C" (shape input) (at 240.03 86.36 180) (fields_autoplaced)
@@
     )
   )
+  (global_label "ATM_RX" (shape input) (at 170.18 91.44 0) (fields_autoplaced)
+    (effects (font (size 1.27 1.27)) (justify left))
+    (property "Intersheet References" "${INTERSHEET_REFS}" (id 0) (at 179.459 91.3606 0)
+      (effects (font (size 1.27 1.27)) (justify left) hide)
+    )
+  )
   (global_label "UARTSW_RX_C" (shape input) (at 240.03 83.82 180) (fields_autoplaced)
     (effects (font (size 1.27 1.27)) (justify right))
     (property "Intersheet References" "${INTERSHEET_REFS}" (id 0) (at 0 0 0)
       (effects (font (size 1.27 1.27)) hide)
+    )
+  )
+  (global_label "ATM_TX" (shape input) (at 153.67 91.44 0) (fields_autoplaced)
+    (effects (font (size 1.27 1.27)) (justify left))
+    (property "Intersheet References" "${INTERSHEET_REFS}" (id 0) (at 162.6466 91.3606 0)
+      (effects (font (size 1.27 1.27)) (justify left) hide)
     )
   )
@@
     (property "Reference" "R304" (id 0) (at 53.34 109.0422 90))
     (property "Value" "2.2k" (id 1) (at 53.34 111.3536 90))
-    (property "Footprint" "Resistor_SMD:R_0603_1608Metric_Pad1.05x0.95mm_HandSolder" (id 2) (at 53.34 112.522 90)
-      (effects (font (size 1.27 1.27)) hide)
-    )
+    (property "Footprint" "Resistor_SMD:R_0603_1608Metric_Pad0.98x0.95mm_HandSolder" (id 2) (at 53.34 112.522 90)
+      (effects (font (size 1.27 1.27)) hide)
+    )
