File: usb_hub.kicad_sch (KiCad schematic)
At the start: 49 parts, among them J201 Conn_02x04_Top_Bottom, J203 Conn_01x04, J204 Conn_01x08, J205 Conn_01x04, J206 Conn_01x04, J207 Conn_01x04, J208 Conn_01x04, U101 LAN9514, U201 SN74CBT3253, U202 PCF8574

Commit message: Add i2c_sampler, update to revision 3
Parts:
- removed J203: Conn_01x04, Connector_PinHeader_2.54mm:PinHeader_1x04_P2.54mm_Vertical, symbol Connector_Generic:Conn_01x04
- removed J204: Conn_01x08, Connector_PinHeader_2.54mm:PinHeader_2x04_P2.54mm_Vertical, symbol Connector_Generic:Conn_01x08
- removed U202: PCF8574, Package_SO:SOIC-16W_7.5x10.3mm_P1.27mm, symbol Interface_Expansion:PCF8574
- added D203: LED, LED_SMD:LED_0603_1608Metric_Pad1.05x0.95mm_HandSolder, symbol Device:LED
- added R224: 470, Resistor_SMD:R_0603_1608Metric_Pad0.98x0.95mm_HandSolder, symbol Device:R
- J202: value (none) -> 8P8C_LED_Shielded; footprint (none) -> Connector_RJ:RJ45_Cetus_J1B1211CCD_Horizontal
- R210, R211: footprint Resistor_SMD:R_0603_1608Metric_Pad1.05x0.95mm_HandSolder -> Resistor_SMD:R_0603_1608Metric_Pad0.98x0.95mm_HandSolder
Connections:
- net +3V3: now also R224.1
- new net: D203.2 (A), R224.2
- new net FDX_LED: D203.1 (K)
