File: iotether.kicad_pcb (KiCad board)
At the start: 2 copper layers, 92 x 100 mm, 181 parts, among them J1 Conn_02x03_Counter_Clockwise, J101 USB_C_Receptacle_USB2.0, J102 Barrel_Jack, J103 Conn_02x04_Odd_Even, J201 Conn_02x04_Top_Bottom, J202 8P8C_LED_Shielded, J205 Conn_01x04, J206 Conn_01x04, J207 Conn_01x04, J208 Conn_01x04, J301 Conn_01x12, J302 Conn_01x12, J303 Conn_01x12, J304 Conn_01x12, J305 Conn_02x04_Odd_Even, J306 Conn_01x09, J307 Conn_01x09, J308 Conn_02x04_Odd_Even, SW1 SW_SPDT, SW301 SW_Push, SW302 SW_Push, SW303 SW_Push, SW304 SW_Push, U101 LAN9514, U102 93CxxC, U103 LM1117-3.3, U104 MCP73831-2-OT, U105 AP62200, U201 SN74CBT3253, U301 FT4232H, U302 93CxxC, U303 ATmega328P-P, U304 FE1.1s, U408 LM75B, U409 DS1307+, Y101 Crystal, Y301 Crystal, Y302 Crystal, Y303 Crystal, Y401 Crystal

Commit message: Update IoTether and I2C sampler
Parts:
- added J104: Conn_01x05, Library:009155003541006, B.Cu at (161.0, 127.4)
Routing:
- net Net-(BT101-Pad1): track 8.83 -> 37.3 mm, vias 0 -> 1
Other:
- board text added: "IoTether Rev. 5.1 2025-07-27 website.peterjin.org/wiki/IoTether"
- board text removed: "IoTether Rev. 5 2025-03-16 website.peterjin.org/wiki/IoTether"
Changed lines of the file:
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@@
       (drillshape 0)
       (scaleselection 1)
-      (outputdirectory "/home/sebastian/Documents/gerbers/")
+      (outputdirectory "/home/sebastian/Documents/gerbers-20250728/")
     )
   )
@@
   (net 183 "unconnected-(J101-PadB8)")
   (net 184 "unconnected-(U105-Pad5)")
+  (net 185 "unconnected-(J104-Pad2)")
   (footprint "Capacitor_SMD:C_0603_1608Metric_Pad1.05x0.95mm_HandSolder" (layer "F.Cu")
     (at 120.375 83.5)
@@
     (property "Sheetname" "")
     (attr through_hole)
-    (fp_text reference "J102" (at -8.45 5.75) (layer "F.SilkS")
+    (fp_text reference "J102" (at 1 6.2) (layer "F.SilkS")
       (effects (font (size 1 1) (thickness 0.15)))
     )
@@
     (property "Sheetname" "")
     (attr through_hole)
-    (fp_text reference "C127" (at 1.9 -5.25 90) (layer "F.SilkS")
+    (fp_text reference "C127" (at 2.628 5.014 90) (layer "F.SilkS")
       (effects (font (size 1 1) (thickness 0.15)))
     )
@@
     )
   )
+  (footprint "Library:009155003541006" (layer "B.Cu")
+    (at 161 127.4 90)
+    (property "Sheetfile" "iotether.kicad_sch")
+    (property "Sheetname" "")
+    (attr smd)
+    (fp_text reference "J104" (at -2.5 3.5 270 unlocked) (layer "B.SilkS")
+      (effects (font (size 1 1) (thickness 0.15)) (justify mirror))
+    )
+    (fp_text value "Conn_01x05" (at 0 -3 270 unlocked) (layer "B.Fab")
+      (effects (font (size 1 1) (thickness 0.15)) (justify mirror))
+    )
+    (fp_text user "${REFERENCE}" (at 0 0 270 unlocked) (layer "B.Fab")
+      (effects (font (size 1 1) (thickness 0.15)) (justify mirror))
+    )
+    (fp_line (start 4.5 2) (end 4.5 1.5) (layer "B.SilkS") (width 0.12))
+    (fp_line (start -4.5 1.5) (end -4.5 2) (layer "B.SilkS") (width 0.12))
+    (fp_line (start -4.5 2) (end -3.5 2) (layer "B.SilkS") (width 0.12))
+    (fp_line (start -4.5 -2) (end -4 -2) (layer "B.SilkS") (width 0.12))
+    (fp_line (start 3.5 2) (end 4.5 2) (layer "B.SilkS") (width 0.12))
+    (fp_line (start -4.5 -1.5) (end -4.5 -2) (layer "B.SilkS") (width 0.12))
+    (fp_line (start 4.5 -2) (end 4.5 -1.5) (layer "B.SilkS") (width 0.12))
+    (fp_line (start 4 -2) (end 4.5 -2) (layer "B.SilkS") (width 0.12))
+    (fp_rect (start -3.5 1.5) (end 3.5 -1.95) (layer "Dwgs.User") (width 0.12) (fill none))
+    (fp_rect (start -4.5 2) (end 4.5 -2) (layer "Dwgs.User") (width 0.12) (fill none))
+    (pad "1" smd roundrect (at -2.5 2.15 90) (size 1.3 1) (layers "B.Cu" "B.Paste" "B.Mask") (roundrect_rratio 0.25)
+      (net 61 "Net-(BT101-Pad1)") (pinfunction "Pin_1") (pintype "passive"))
+    (pad "2" smd roundrect (at 0 2.15 90) (size 1.3 1) (layers "B.Cu" "B.Paste" "B.Mask") (roundrect_rratio 0.25)
+      (net 185 "unconnected-(J104-Pad2)") (pinfunction "Pin_2") (pintype "passive"))
+    (pad "3" smd roundrect (at 2.5 2.15 90) (size 1.3 1) (layers "B.Cu" "B.Paste" "B.Mask") (roundrect_rratio 0.25)
+      (net 1 "GND") (pinfunction "Pin_3") (pintype "passive"))
+    (pad "4" smd roundrect (at -4.4 0 90) (size 1.5 2.15) (layers "B.Cu" "B.Paste" "B.Mask") (roundrect_rratio 0.25)
+      (net 1 "GND") (pinfunction "Pin_4") (pintype "passive") (zone_connect 2))
+    (pad "5" smd roundrect (at 4.4 0 90) (size 1.5 2.15) (layers "B.Cu" "B.Paste" "B.Mask") (roundrect_rratio 0.25)
+      (net 1 "GND") (pinfunction "Pin_5") (pintype "passive") (zone_connect 2))
+    (zone (net 0) (net_name "") (layers "B.Cu" "Dwgs.User") (hatch edge 0.508)
+      (connect_pads (clearance 0))
+      (min_thickness 0.254)
+      (keepout (tracks not_allowed) (vias not_allowed) (pads not_allowed) (copperpour not_allowed) (footprints allowed))
+      (fill (thermal_gap 0.508) (thermal_bridge_width 0.508))
+      (polygon
+        (pts
+          (xy 162.5 130.9)
+          (xy 162.5 123.9)
+          (xy 159.05 123.9)
+          (xy 159.05 130.9)
+        )
+      )
+    )
+  )
   (footprint "Resistor_SMD:R_0603_1608Metric_Pad0.98x0.95mm_HandSolder" (layer "B.Cu")
     (at 136.1875 60.8)
@@
   (gr_line (start 167 50) (end 167 150) (layer "Edge.Cuts") (width 0.05))
   (gr_line (start 167 150) (end 75 150) (layer "Edge.Cuts") (width 0.05))
-  (gr_text "IoTether Rev. 5 2025-03-16\nwebsite.peterjin.org/wiki/IoTether" (at 103 140.75) (layer "F.SilkS")
+  (gr_text "IoTether Rev. 5.1 2025-07-27\nwebsite.peterjin.org/wiki/IoTether" (at 103 140.75) (layer "F.SilkS")
     (effects (font (size 1 1) (thickness 0.25)))
   )
+  (dimension (type aligned) (layer "B.SilkS")
+    (pts (xy 157.988 137.16) (xy 157.988 130))
+    (height 0)
+    (gr_text "7.1600 mm" (at 157.25 133.75 90) (layer "B.SilkS")
+      (effects (font (size 0.5 0.5) (thickness 0.1)) (justify mirror))
+    )
+    (format (units 3) (units_format 1) (precision 4))
+    (style (thickness 0.12) (arrow_length 1.27) (text_position_mode 2) (extension_height 0.58642) (extension_offset 0.5) keep_text_aligned)
+  )
+  (dimension (type aligned) (layer "B.SilkS")
+    (pts (xy 81.788 137.16) (xy 157.988 137.16))
+    (height 0)
+    (gr_text "76.2000 mm" (at 119.888 136.01) (layer "B.SilkS")
+      (effects (font (size 1 1) (thickness 0.15)) (justify mirror))
+    )
+    (format (units 3) (units_format 1) (precision 4))
+    (style (thickness 0.12) (arrow_length 1.27) (text_position_mode 0) (extension_height 0.58642) (extension_offset 0.5) keep_text_aligned)
+  )
   (segment (start 114.75 84) (end 114.75 80.5) (width 0.25) (layer "F.Cu") (net 1))
   (segment (start 114.75 86) (end 114.75 84) (width 0.25) (layer "F.Cu") (net 1))
@@
   (segment (start 120 98.75) (end 119.25 99.5) (width 0.25) (layer "B.Cu") (net 56))
   (segment (start 122.625 97.5) (end 122.25 97.5) (width 0.25) (layer "B.Cu") (net 56))
+  (segment (start 166 130.75) (end 165.25 130) (width 0.5) (layer "F.Cu") (net 61))
+  (segment (start 153.25 140.25) (end 165.5 140.25) (width 0.5) (layer "F.Cu") (net 61))
   (segment (start 150.495 141.605) (end 150.495 145.0975) (width 0.5) (layer "F.Cu") (net 61))
+  (segment (start 166 139.75) (end 166 130.75) (width 0.5) (layer "F.Cu") (net 61))
+  (segment (start 165.5 140.25) (end 166 139.75) (width 0.5) (layer "F.Cu") (net 61))
+  (segment (start 150.495 141.605) (end 151.895 141.605) (width 0.5) (layer "F.Cu") (net 61))
+  (segment (start 151.895 141.605) (end 153.25 140.25) (width 0.5) (layer "F.Cu") (net 61))
   (segment (start 150.495 145.0975) (end 149.86 145.7325) (width 0.5) (layer "F.Cu") (net 61))
+  (via (at 165.25 130) (size 0.8) (drill 0.4) (layers "F.Cu" "B.Cu") (net 61))
   (segment (start 146.345 143.505) (end 147.6325 143.505) (width 0.5) (layer "B.Cu") (net 61))
+  (segment (start 165.15 129.9) (end 165.25 130) (width 0.5) (layer "B.Cu") (net 61))
+  (segment (start 163.15 129.9) (end 165.15 129.9) (width 0.5) (layer "B.Cu") (net 61))
   (segment (start 147.6325 143.505) (end 149.86 145.7325) (width 0.5) (layer "B.Cu") (net 61))
   (segment (start 154.94 144.35) (end 154.305 144.985) (width 0.25) (layer "F.Cu") (net 62))
@@
       )
     )
+  )
+  (zone (net 0) (net_name "") (layer "B.Cu") (hatch edge 0.508)
+    (connect_pads (clearance 0))
+    (min_thickness 0.254)
+    (keepout (tracks not_allowed) (vias not_allowed) (pads not_allowed) (copperpour not_allowed) (footprints allowed))
+    (fill (thermal_gap 0.508) (thermal_bridge_width 0.508))
+    (polygon
+      (pts
+        (xy 159.75 131)
+        (xy 157.5 131)
+        (xy 157.5 127.75)
+        (xy 159.75 127.75)
+      )
+    )
