File: iotether.kicad_sch (KiCad schematic)
At the start: 70 parts, among them J1 Conn_02x03_Counter_Clockwise, J101 USB_C_Receptacle_USB2.0, J102 Barrel_Jack, J103 Conn_02x04_Odd_Even, SW1 SW_SPDT, U101 LAN9514, U102 93CxxC, U103 LM1117-3.3, U104 MCP73831-2-OT, U105 AP62200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

Commit message: Update IoTether and I2C sampler
Parts:
- added J104: Conn_01x05, Library:009155003541006, symbol Connector_Generic:Conn_01x05
Connections:
- net GND: now also J104.3 (Pin_3), J104.4 (Pin_4), J104.5 (Pin_5)
- net at BT101.1 (+), C125.1, U104.3 (VBAT): now also J104.1 (Pin_1)
Changed lines of the file:
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@@
   (junction (at 198.12 22.86) (diameter 0) (color 0 0 0 0)
   )
+  (junction (at 148.59 189.23) (diameter 0) (color 0 0 0 0)
+  )
   (junction (at 205.74 30.48) (diameter 0) (color 0 0 0 0)
   )
@@
   (junction (at 152.4 30.48) (diameter 0) (color 0 0 0 0)
   )
+  (junction (at 132.08 179.07) (diameter 0) (color 0 0 0 0)
+  )
   (junction (at 22.86 55.88) (diameter 0) (color 0 0 0 0)
   )
@@
   (junction (at 104.14 83.82) (diameter 0) (color 0 0 0 0)
   )
+  (junction (at 148.59 186.69) (diameter 0) (color 0 0 0 0)
+  )
   (junction (at 52.07 102.87) (diameter 0) (color 0 0 0 0)
   )
+  (junction (at 132.08 186.69) (diameter 0) (color 0 0 0 0)
+  )
   (junction (at 27.94 60.96) (diameter 0) (color 0 0 0 0)
   )
@@
     (stroke (width 0) (type default) (color 0 0 0 0))
   )
+  (wire (pts (xy 148.59 189.23) (xy 148.59 191.77))
+    (stroke (width 0) (type default) (color 0 0 0 0))
+  )
   (wire (pts (xy 134.62 69.85) (xy 134.62 76.2))
     (stroke (width 0) (type default) (color 0 0 0 0))
@@
     (stroke (width 0) (type default) (color 0 0 0 0))
   )
+  (wire (pts (xy 148.59 179.07) (xy 132.08 179.07))
+    (stroke (width 0) (type default) (color 0 0 0 0))
+  )
   (wire (pts (xy 71.12 80.01) (xy 66.04 80.01))
     (stroke (width 0) (type default) (color 0 0 0 0))
@@
     (stroke (width 0) (type default) (color 0 0 0 0))
   )
+  (wire (pts (xy 148.59 181.61) (xy 148.59 179.07))
+    (stroke (width 0) (type default) (color 0 0 0 0))
+  )
   (wire (pts (xy 218.44 22.86) (xy 226.06 22.86))
     (stroke (width 0) (type default) (color 0 0 0 0))
@@
     (stroke (width 0) (type default) (color 0 0 0 0))
   )
+  (wire (pts (xy 148.59 186.69) (xy 148.59 189.23))
+    (stroke (width 0) (type default) (color 0 0 0 0))
+  )
   (wire (pts (xy 45.72 22.86) (xy 45.72 25.4))
     (stroke (width 0) (type default) (color 0 0 0 0))
@@
     (stroke (width 0) (type default) (color 0 0 0 0))
   )
+  (wire (pts (xy 132.08 186.69) (xy 148.59 186.69))
+    (stroke (width 0) (type default) (color 0 0 0 0))
+  )
   (global_label "UP_D+" (shape input) (at 82.55 34.29 0) (fields_autoplaced)
     (effects (font (size 1.27 1.27)) (justify left))
@@
     (pin "2")
   )
+  (symbol (lib_id "Connector_Generic:Conn_01x05") (at 153.67 186.69 0) (unit 1)
+    (in_bom yes) (on_board yes) (fields_autoplaced)
+    (property "Reference" "J104" (id 0) (at 156.21 185.4199 0)
+      (effects (font (size 1.27 1.27)) (justify left))
+    )
+    (property "Value" "Conn_01x05" (id 1) (at 156.21 187.9599 0)
+      (effects (font (size 1.27 1.27)) (justify left))
+    )
+    (property "Footprint" "Library:009155003541006" (id 2) (at 153.67 186.69 0)
+      (effects (font (size 1.27 1.27)) hide)
+    )
+    (property "Datasheet" "~" (id 3) (at 153.67 186.69 0)
+      (effects (font (size 1.27 1.27)) hide)
+    )
+    (pin "1")
+    (pin "2")
+    (pin "3")
+    (pin "4")
+    (pin "5")
+  )
   (symbol (lib_id "Device:L") (at 165.1 130.81 90) (unit 1)
     (in_bom yes) (on_board yes) (fields_autoplaced)
@@
       (reference "J103") (unit 1) (value "Conn_02x04_Odd_Even") (footprint "Connector_PinHeader_2.54mm:PinHeader_2x04_P2.54mm_Vertical")
     )
+    (path "/315f3242-1e65-4cf8-b76e-5d6f48cd973b"
+      (reference "J104") (unit 1) (value "Conn_01x05") (footprint "Library:009155003541006")
+    )
     (path "/00000000-0000-0000-0000-000061b77588/00000000-0000-0000-0000-000061bb5af3"
