File: i2c_sampler/i2c_sampler/i2c_sampler.kicad_pcb (KiCad board)
At the start: 2 copper layers, 75 x 50 mm, 55 parts, among them J1 Conn_01x04, J10 Conn_01x03, J11 Conn_01x03, J12 Barrel_Jack_Switch, J13 Conn_01x04, J2 Conn_01x03, J3 Conn_01x03, J4 Conn_01x03, J5 Conn_01x03, J6 Conn_01x03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

Commit message: Update I2C sampler and IoTether, add voltage converter
Parts:
- added D4: BAT54A, Package_TO_SOT_SMD:SOT-23, B.Cu at (74.0, 89.8)
- added R12: R, Resistor_SMD:R_0603_1608Metric, B.Cu at (71.4, 88.5)
- added R13: R, Resistor_SMD:R_0603_1608Metric, B.Cu at (111.3, 72.1)
Connections:
- U7 pad 5: Net-(C11-Pad1) -> Net-(U7-Pad5)
Routing:
- net Net-(C11-Pad1): track 34.3 -> 25.2 mm
- net VDD: track 298.0 -> 300.2 mm
- net Net-(U7-Pad5): track 0.00 -> 2.17 mm
- net Net-(D4-Pad1): track 0.00 -> 1.79 mm
- net Net-(BT1-Pad1): track 17.1 -> 18.5 mm
Other:
- board text added: "website.peterjin.org/wiki/I2C_Sampler Rev 2 2024-04-06"
- board text removed: "website.peterjin.org/wiki/I2C_Sampler"

Commit message: Update IoTether and I2C sampler
Parts:
- added C13: C, Capacitor_SMD:C_0805_2012Metric, F.Cu at (105.5, 64.0)
- added C14: C, Capacitor_SMD:C_0805_2012Metric, F.Cu at (105.5, 76.8)
- added C15: C, Capacitor_SMD:C_0805_2012Metric, F.Cu at (106.5, 56.7)
- added C16: C, Capacitor_SMD:C_0805_2012Metric, B.Cu at (102.5, 75.0)
- added D5: LED, LED_SMD:LED_0603_1608Metric, F.Cu at (103.2, 51.6)
- added D6: LED, LED_SMD:LED_0603_1608Metric, F.Cu at (103.5, 81.3)
- added J14: Conn_01x09, Connector_USB:USB_A_Wuerth_61400826021_Horizontal_Stacked, F.Cu at (93.7, 58.6)
- added J15: Conn_01x05, Library:009155003541006, F.Cu at (102.2, 58.0)
- added J16: Conn_01x05, Library:009155003541006, B.Cu at (98.0, 81.3)
- added R14: R, Resistor_SMD:R_0603_1608Metric, F.Cu at (111.4, 51.8)
- added R15: R, Resistor_SMD:R_0603_1608Metric, F.Cu at (104.8, 79.0)
- added R16: R, Resistor_SMD:R_0603_1608Metric, B.Cu at (105.8, 51.8)
- added R17: R, Resistor_SMD:R_0603_1608Metric, B.Cu at (103.5, 84.3)
- added U8: MCP73831-2-OT, Package_TO_SOT_SMD:SOT-23-5, F.Cu at (106.9, 53.0)
- added U9: MCP73831-2-OT, Package_TO_SOT_SMD:SOT-23-5, B.Cu at (103.0, 80.6)
Routing:
- net VDD: track 300.2 -> 364.1 mm, vias 12 -> 14
- net Net-(C16-Pad1): track 0.00 -> 12.3 mm, vias 0 -> 2
- net Net-(D5-Pad2): track 0.00 -> 5.09 mm, vias 0 -> 1
- net Net-(D6-Pad2): track 0.00 -> 4.96 mm, vias 0 -> 1
- net Net-(C15-Pad1): track 0.00 -> 4.29 mm
- net GND: track 55.6 -> 58.9 mm, vias 8 -> 21
- net Net-(D6-Pad1): track 0.00 -> 3.24 mm, vias 0 -> 1
- net Net-(R15-Pad1): track 0.00 -> 2.06 mm, vias 0 -> 1
- net Net-(J14-Pad6): track 0.00 -> 2.00 mm
- net Net-(J14-Pad2): track 0.00 -> 2.00 mm
- net Net-(D5-Pad1): track 0.00 -> 1.92 mm
- net Net-(R14-Pad1): track 0.00 -> 1.85 mm
- added copper zone on F.Cu, net GND
Other:
- board text added: "website.peterjin.org/wiki/I2C_Sampler Rev 3 2025-07-28"
- board text removed: "website.peterjin.org/wiki/I2C_Sampler Rev 2 2024-04-06"
